File: mezzanine-board/sensorPCB.kicad_sch (KiCad schematic)
At the start: 22 parts, among them J1 SFMC-105-01-L-D, U1 AS72651, U2 4MB Flash, U3 AS72652, U4 AS72653

Commit message: Initial Routing
Connections:
- net CSN_EE: now also J1.1; no longer J1.5
- net GND: now also J1.10; no longer J1.6
- net INT: now also J1.6; no longer J1.10
- net RESN: now also J1.9; no longer J1.4
- net RX/SCL: now also J1.2; no longer J1.7
- net SPI_MOSI: now also J1.5; no longer J1.1
- net SPI_SCK: now also J1.7; no longer J1.2
- net TX/SDA: now also J1.4; no longer J1.9

Commit message: Update larger board design
Parts:
- H1, H2: footprint Mounting_Wuerth:Mounting_Wuerth_WA-SMSI-M2.5_H0.5mm_9774005151 -> MountingHole:MountingHole_2.7mm_M2.5
Connections:
- net at D1.2 (A): now also U1.18 (LED_IND); no longer U1.15 (LED_DRV)
Other:
- moved on the sheet: D1
Changed lines of the file:
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@@
 	)
 	(no_connect
-		(at 66.04 54.61)
-	)
-	(no_connect
 		(at 232.41 90.17)
 	)
@@
 		(at 232.41 49.53)
 	)
+	(no_connect
+		(at 74.93 57.15)
+	)
 	(wire
 		(pts
@@
 	(wire
 		(pts
-			(xy 66.04 54.61) (xy 74.93 54.61)
-		)
-		(stroke
-			(width 0)
-			(type default)
-		)
-	)
-	(wire
-		(pts
 			(xy 158.75 44.45) (xy 166.37 44.45)
 		)
@@
 	(wire
 		(pts
+			(xy 60.96 54.61) (xy 74.93 54.61)
+		)
+		(stroke
+			(width 0)
+			(type default)
+		)
+	)
+	(wire
+		(pts
 			(xy 30.48 50.8) (xy 20.32 50.8)
 		)
@@
 	(wire
 		(pts
-			(xy 60.96 57.15) (xy 74.93 57.15)
-		)
-		(stroke
-			(width 0)
-			(type default)
-		)
-	)
-	(wire
-		(pts
 			(xy 271.78 93.98) (xy 276.86 93.98)
 		)
@@
 	(wire
 		(pts
-			(xy 48.26 57.15) (xy 53.34 57.15)
+			(xy 48.26 54.61) (xy 53.34 54.61)
 		)
 		(stroke
@@
 			)
 		)
-		(property "Footprint" "Mounting_Wuerth:Mounting_Wuerth_WA-SMSI-M2.5_H0.5mm_9774005151"
+		(property "Footprint" "MountingHole:MountingHole_2.7mm_M2.5"
 			(at 25.4 101.6 0)
 			(hide yes)
@@
 	(symbol
 		(lib_id "Device:LED")
-		(at 57.15 57.15 0)
+		(at 57.15 54.61 0)
 		(unit 1)
 		(body_style 1)
@@
 		(dnp no)
 		(property "Reference" "D1"
-			(at 57.15 52.578 0)
+			(at 57.15 50.038 0)
 			(show_name no)
 			(do_not_autoplace no)
@@
 		)
 		(property "Value" "GREEN"
-			(at 57.15 54.61 0)
+			(at 57.15 52.07 0)
 			(show_name no)
 			(do_not_autoplace no)
@@
 		)
 		(property "Footprint" "LED_SMD:LED_0603_1608Metric"
-			(at 57.658 61.214 0)
+			(at 57.658 58.674 0)
 			(show_name no)
 			(do_not_autoplace no)
@@
 		)
 		(property "Datasheet" ""
-			(at 57.15 57.15 0)
+			(at 57.15 54.61 0)
 			(hide yes)
 			(show_name no)
@@
 		)
 		(property "Description" "Light emitting diode"
-			(at 57.15 57.15 0)
+			(at 57.15 54.61 0)
 			(hide yes)
 			(show_name no)
@@
 		)
 		(property "Sim.Pins" "1=K 2=A"
-			(at 57.15 57.15 0)
+			(at 57.15 54.61 0)
 			(hide yes)
 			(show_name no)
@@
 			)
 		)
-		(property "Footprint" "Mounting_Wuerth:Mounting_Wuerth_WA-SMSI-M2.5_H0.5mm_9774005151"
+		(property "Footprint" "MountingHole:MountingHole_2.7mm_M2.5"
 			(at 25.4 109.22 0)
 			(hide yes)
@@
 	(symbol
 		(lib_id "power:+3.3V")
-		(at 48.26 57.15 0)
+		(at 48.26 54.61 0)
 		(unit 1)
 		(body_style 1)
@@
 		(fields_autoplaced yes)
 		(property "Reference" "#PWR03"
-			(at 48.26 60.96 0)
+			(at 48.26 58.42 0)
 			(hide yes)
 			(show_name no)
@@
 		)
 		(property "Value" "+3.3V"
-			(at 48.26 52.07 0)
+			(at 48.26 49.53 0)
 			(show_name no)
 			(do_not_autoplace no)
@@
 		)
 		(property "Footprint" ""
-			(at 48.26 57.15 0)
+			(at 48.26 54.61 0)
 			(hide yes)
 			(show_name no)
@@
 		)
 		(property "Datasheet" ""
-			(at 48.26 57.15 0)
+			(at 48.26 54.61 0)
 			(hide yes)
 			(show_name no)
@@
 		)
 		(property "Description" "Power symbol creates a global label with name \"+3.3V\""
-			(at 48.26 57.15 0)
+			(at 48.26 54.61 0)
 			(hide yes)
 			(show_name no)

Commit message: Moved RA connectors back to 16mm away
Connections:
- net SLV1_RESN: no longer U4.2 (RESN)
- net SLV2_RESN: now also U4.2 (RESN)
Changed lines of the file:
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@@
-		)
-	)
-	(label "SLV1_RESN"
-		(at 232.41 74.93 180)
-		(effects
-			(font
-				(size 1.27 1.27)
-			)
-			(justify right bottom)
 		)
 	)
@@
 		)
 	)
+	(label "SLV2_RESN"
+		(at 232.41 74.93 180)
+		(effects
+			(font
+				(size 1.27 1.27)
+			)
+			(justify right bottom)
+		)
+	)
