File: main-board/StackInterface.kicad_sch (KiCad schematic)
At the start: 2 parts

Commit message: Update larger board design
Connections:
- net 5V_PERM renamed +5V
- no-connect marks 97 -> 99
Other:
- moved on the sheet: H1

Commit message: Update PCB designs, CAD assemblies, analysis and BOM files
Connections:
- net UART_A_DN renamed STACK TX
- net UART_A_UP renamed STACK RX
- no-connect marks 99 -> 95
